Commit message: I have fixed the .xacro file for the .urdf file. I now need to fix the meshes.

File: abb_irb1600_support/urdf/irb1600_6_12_macro_original.xacro (robot description, xacro)
@@ -137,5 +137,6 @@
   <joint name="${prefix}joint_3" type="revolute">
     <!-- According to the spec sheet, this is the correct value for the 1.45 meter version. -->
-    <origin xyz="0 0 0.700" rpy="0 0 0"/>
+    <!-- <origin xyz="0 0 0.700" rpy="0 0 0"/> -->
+    <origin xyz="0 0 0.475" rpy="0 0 0"/>
     <!-- This is the original line. It contains the "z" value for the 1.2 meter version of the abb irb 1600 -->
     <!-- <origin xyz="0 0 0.475" rpy="0 0 0"/> -->
